File: EAGLE/projects/Bot/bot.brd (EAGLE design)
At the start: 124.3 x 90 mm, 17 parts, among them IC1 7805T, U3 ARDUINO_SHIELDLABEL

Commit message: Final PCB
PCB
Parts:
- added JP2: (no value), pinhead:1X02
- R5: value 1k -> 10
- moved C2 82.6 mm to (83.8, 91.4), turned to 0 degrees
- moved C1 77.1 mm to (83.8, 85.1), turned to 0 degrees
- moved R1 71.7 mm to (69.8, 91.4), flipped to the top, turned to 0 degrees
- moved LED2 70.3 mm to (102.9, 78.7)
- moved LED1 68.3 mm to (102.9, 88.9)
- moved R5 68.0 mm to (69.8, 80.0)
- moved R4 67.9 mm to (69.8, 83.8)
- moved R3 64.9 mm to (69.8, 87.6), flipped to the top
- moved R2 64.2 mm to (69.8, 76.2)
- moved U$1 64.1 mm to (116.8, 85.1), turned to 270 degrees
- moved U$2 59.1 mm to (116.8, 66.0)
- moved TXS0108E1:JP1 57.4 mm to (76.2, 72.4), turned to 0 degrees
- moved TXS0108E1:JP2 44.4 mm to (76.2, 59.7), flipped to the top, turned to 180 degrees
- moved U3 29.3 mm to (120.7, 2.54)
- moved PI 5.96 mm to (1.27, 30.5)
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Connections:
- removed net S$1: IC1.2
- net 0: now also IC1.2, JP2.1, JP7.2
- net PWR+: now also JP2.2
Routing:
- net L_US_ECHO: track 183.1 -> 42.7 mm
- net 0: track 187.2 -> 322.5 mm
- net R_SPD: track 0.00 -> 102.3 mm
- net L_SPD: track 0.00 -> 86.1 mm
- net PWR+: track 116.3 -> 180.9 mm
- net N$16: track 0.00 -> 62.2 mm
- net N$1: track 0.00 -> 51.6 mm
- net N$14: track 22.6 -> 60.2 mm
- net L_BCK: track 0.00 -> 36.2 mm
- net R_BCK: track 0.00 -> 33.5 mm
- net L_FWD: track 0.00 -> 33.4 mm
- net N$15: track 40.6 -> 73.1 mm
- net PI_3V3: track 43.1 -> 74.8 mm
- net R_FWD: track 0.00 -> 19.9 mm
- net N$13: track 39.4 -> 57.2 mm
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Other:
- board size 124.3 x 90 mm -> 123.2 x 96.2 mm

Commit message: Almost error free
.
Parts:
- moved R2 0.63 mm to (69.9, 76.8)
Routing:
- net PWR+: track 180.9 -> 218.3 mm
- net N$14: track 60.2 -> 85.1 mm
- net R_BCK: track 33.5 -> 54.6 mm
- net R_US_ECHO: track 44.9 -> 64.0 mm
- net N$15: track 73.1 -> 60.6 mm
- net N$13: track 57.2 -> 67.1 mm
- net L_SPD: track 86.1 -> 92.9 mm
- net R_SPD: track 102.3 -> 107.9 mm
- net PI_5V: track 192.8 -> 189.1 mm
- net L_FWD: track 33.4 -> 36.4 mm
- net 0: track 322.5 -> 325.0 mm
- net PI_3V3: track 74.8 -> 76.5 mm
Other:
- board size 123.2 x 96.2 mm -> 122.1 x 96.2 mm

Commit message: Ready to mill
Parts:
- added KK1: SK129-PAD, heatsink:SK129
- moved JP2 51.5 mm to (57.8, 18.5), turned to 90 degrees
- moved R1 16.1 mm to (85.1, 86.4)
- moved C2 15.3 mm to (85.1, 76.2)
- moved LED2 14.0 mm to (104.1, 64.8)
- moved LED1 8.98 mm to (104.1, 80.0)
- moved C1 4.02 mm to (85.1, 81.3)
- moved U$1 3.81 mm to (116.8, 81.3), turned to 90 degrees
- moved IC1 3.63 mm to (31.8, 20.3)
- moved PI 2.84 mm to (0.00, 27.9)
- moved R3 2.54 mm to (69.8, 90.2)
- moved TXS0108E1:JP1 2.54 mm to (76.2, 69.8), turned to 180 degrees
- moved TXS0108E1:JP2 2.54 mm to (76.2, 57.1), turned to 0 degrees
- moved JP7 1.94 mm to (5.08, 19.1)
- moved R2 1.90 mm to (69.8, 74.9)
- moved R4 1.27 mm to (69.8, 85.1)
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Routing:
- net R_BCK: track 54.6 -> 113.9 mm, vias 0 -> 1
- net R_FWD: track 20.1 -> 70.2 mm, vias 0 -> 2
- net PI_5V: track 189.1 -> 153.7 mm, vias 0 -> 1
- net N$14: track 85.1 -> 57.4 mm
- net N$1: track 51.9 -> 28.2 mm
- net N$15: track 60.6 -> 82.5 mm
- net L_US_ECHO: track 42.8 -> 64.5 mm
- net 0: track 325.0 -> 305.3 mm, vias 0 -> 1
- net R_SPD: track 107.9 -> 89.4 mm
- net N$2: track 45.8 -> 62.2 mm, vias 0 -> 1
- net PI_3V3: track 76.5 -> 63.1 mm
- net R_US_TRIG: track 68.8 -> 80.7 mm
- net L_BCK: track 36.2 -> 24.7 mm
- net N$13: track 67.1 -> 56.0 mm
- net L_SPD: track 92.9 -> 103.1 mm
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- added copper zone on layer 16, net GND
Other:
- board size 122.1 x 96.2 mm -> 121.9 x 93.7 mm
