File: EAGLE/projects/Bot/Evan_bot.brd (EAGLE design)
At the start: 122.5 x 95 mm, 22 parts, among them IC1 7805T, U3 ARDUINO_SHIELDLABEL

Commit message: git
Parts:
- removed S1: (no value), switch:MS243
- moved IC1 90.7 mm to (95.2, 83.4)
- moved KK1 90.7 mm to (95.2, 75.7)
- moved U3 70.5 mm to (62.4, 1.19), turned to 0 degrees
- moved R4 69.3 mm to (18.3, 24.4)
- moved R1 61.9 mm to (42.1, 23.4)
- moved R6 56.5 mm to (55.6, 24.0), turned to 270 degrees
- moved LED1 56.0 mm to (33.3, 8.79)
- moved LED2 56.0 mm to (22.9, 8.89)
- moved R2 56.0 mm to (14.0, 23.9)
- moved U$2 56.0 mm to (10.0, 6.22)
- moved U$1 56.0 mm to (47.6, 6.32)
- moved C1 53.0 mm to (62.7, 78.4), turned to 0 degrees
- moved C2 53.0 mm to (62.7, 69.3), turned to 180 degrees
- moved R5 49.3 mm to (29.7, 23.4)
- moved R3 48.5 mm to (48.0, 23.2)
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Connections:
- removed net N$3: JP2.1, S1.1
- net 0: now also JP2.1; no longer S1.2
Routing:
- net PWR+: track 235.2 -> 69.3 mm
- net R_FWD: track 162.4 -> 0.00 mm, vias 2 -> 0
- net N$4: track 34.5 -> 162.4 mm, vias 2 -> 0
- net L_US_ECHO: track 79.6 -> 206.8 mm, vias 2 -> 0
- net 0: track 468.5 -> 562.5 mm
- net R_SPD: track 91.6 -> 0.00 mm, vias 2 -> 0
- net L_US_TRIG: track 86.7 -> 0.00 mm, vias 2 -> 0
- net R_BCK: track 83.7 -> 0.00 mm, vias 2 -> 0
- net PI_3V3: track 120.1 -> 56.5 mm
- net L_BCK: track 54.3 -> 0.00 mm, vias 2 -> 0
- net PI_5V: track 305.1 -> 254.0 mm
- net R_US_TRIG: track 50.6 -> 0.00 mm, vias 2 -> 0
- net L_FWD: track 49.9 -> 0.00 mm, vias 2 -> 0
- net L_SPD: track 49.2 -> 0.00 mm, vias 2 -> 0
- net N$6: track 52.3 -> 8.78 mm, vias 2 -> 0
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- added copper zone on layer 16, net N$3
- removed copper zone on layer 16, net 0
Other:
- board size 122.5 x 95 mm -> 122 x 94.9 mm
