File: EAGLE/projects/Bot/bot.sch (EAGLE design)
At the start: 17 parts, among them IC1 7805T, U3 ARDUINO_SHIELDLABEL, X1 RASPI_GPIO_B+_PIN

Commit message: revert eagle files
Parts:
- removed JP1, JP5, JP6: (no value), pinhead:PINHD-1X2
- removed JP3, JP4: (no value), pinhead:PINHD-1X4
- removed JP8, JP9: (no value), pinhead:PINHD-1X10
- removed X1: RASPI_GPIO_B+_PIN, raspberrypi_bastelstube_v13:RASPI_GPIO_B+_PIN
- added C1: 330n, rcl:C-US025-025X050
- added C2: 100n, rcl:C-US025-025X050
- added LED1, LED2: (no value), led:LED5MM
- added U$1, U$2: ULTRASONIC-HC-SR04#V, diy-modules:ULTRASONIC-HC-SR04#V
- added X2: RASPI_BOARD_B+_FP, raspberrypi_bastelstube_v13:RASPI_BOARD_B+_FP
- JP7: value VCC -> SHIELD_PWR
Connections:
- removed net N$10: JP9.4, U3.D8
- removed net N$11: JP9.3, U3.*D9
- removed net N$12: JP9.2
- removed net N$17: JP8.4
- removed net N$18: JP8.5
- removed net N$22: JP8.9
- removed net N$4: JP9.9
- removed net N$6: JP9.8, U3.D4
- removed net N$7: JP9.7
- removed net N$8: JP9.6
- removed net N$9: JP9.5, U3.D7
- removed net RPI_PWR+: IC1.VO, JP1.1
- new net B1: JP2.9
- new net B2: JP2.8
- new net B3: JP2.7
- new net B4: JP2.6
- new net B5: JP2.5
- new net B6: JP2.4
- new net B7: JP2.3
- new net B8: JP2.2
- new net GND: JP2.1
- new net N$13: U3.D4
- new net N$14: U3.D7
- new net N$16: U3.*D9
- new net VB: JP2.10
- net 0: now also C1.2, C2.2, U$1.GND, U$2.GND, X2.GND; no longer JP1.2, JP3.4, JP4.4, JP9.1, X1.GND
- net L_BCK: now also X2.GPIO21; no longer JP8.7, X1.GPIO21
- net L_FWD: now also X2.GPIO20; no longer JP8.6, X1.GPIO20
- net L_SPD: now also X2.GPIO12; no longer X1.GPIO12
- net L_US_ECHO: now also X2.GPIO24; no longer X1.GPIO24
- net L_US_TRIG: now also U$1.TRIG, X2.GPIO23; no longer JP3.2, X1.GPIO23
- net N$1: now also U$1.ECHO; no longer JP3.3
- net N$15: now also U3.D8; no longer JP8.2
- net N$2: now also U$2.ECHO; no longer JP4.3
- net N$5: now also LED1.C, LED2.C; no longer JP5.2, JP6.2
- net PI_3V3: now also X2.3V3; no longer JP8.1, JP8.10, X1.3V3
- net PI_5V: now also C2.1, IC1.VO, U$1.VCC, U$2.VCC, X2.5V0; no longer JP3.1, JP4.1, JP9.10, X1.5V0
- net PWR+: now also C1.1, LED1.A, LED2.A; no longer JP5.1, JP6.1
- net R_BCK: now also X2.GPIO06; no longer JP8.8, X1.GPIO06
- net R_FWD: now also X2.GPIO05; no longer JP8.3, X1.GPIO05
- net R_SPD: now also X2.GPIO13; no longer X1.GPIO13
- net R_US_ECHO: now also X2.GPIO22; no longer X1.GPIO22
- net R_US_TRIG: now also U$2.TRIG, X2.GPIO27; no longer JP4.2, X1.GPIO27
Other:
- note removed: "A1"
- note removed: "A2"
- note removed: "A3"
- note removed: "A4"
- note removed: "A5"
- note removed: "A6"
- note removed: "A7"
- note removed: "A8"
- note removed: "B1"
- note removed: "B2"
- note removed: "B3"
- note removed: "B4"
- note removed: "B5"
- note removed: "B6"
- note removed: "B7"
- note removed: "B8"
- note removed: "GND"
- note removed: "OE"
- note removed: "RPI_PWR+"
- note removed: "RPI_PWR-"
- note removed: "VA"
- note removed: "VB"
- moved on the sheet: IC1, JP2, JP7, R1, R2, R3, R4, R5, U3

Commit message: Not finished routing
Not finished routing
Parts:
- removed X2: RASPI_BOARD_B+_FP, raspberrypi_bastelstube_v13:RASPI_BOARD_B+_FP
- added PI: RASPI_BOARD_B+_F, raspberrypi_bastelstube_v13:RASPI_BOARD_B+_F
Connections:
- net 0: now also PI.GND; no longer X2.GND
- net L_BCK: now also PI.GPIO21; no longer X2.GPIO21
- net L_FWD: now also PI.GPIO20; no longer X2.GPIO20
- net L_SPD: now also PI.GPIO12; no longer X2.GPIO12
- net L_US_ECHO: now also PI.GPIO24; no longer X2.GPIO24
- net L_US_TRIG: now also PI.GPIO23; no longer X2.GPIO23
- net PI_3V3: now also PI.3V3; no longer X2.3V3
- net PI_5V: now also PI.5V0; no longer X2.5V0
- net R_BCK: now also PI.GPIO06; no longer X2.GPIO06
- net R_FWD: now also PI.GPIO05; no longer X2.GPIO05
- net R_SPD: now also PI.GPIO13; no longer X2.GPIO13
- net R_US_ECHO: now also PI.GPIO22; no longer X2.GPIO22
- net R_US_TRIG: now also PI.GPIO27; no longer X2.GPIO27

Commit message: Final PCB
PCB
Parts:
- R5: value 1k -> 10
Changed lines of the file:
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@@
 <setting verticaltext="up"/>
 </settings>
-<grid distance="1" unitdist="mm" unit="mm" style="lines" multiple="1" display="yes" altdistance="0.01" altunitdist="inch" altunit="mm"/>
+<grid distance="0.1" unitdist="inch" unit="inch" style="lines" multiple="1" display="no" altdistance="0.01" altunitdist="inch" altunit="inch"/>
 <layers>
 <layer number="1" name="Top" color="4" fill="1" visible="yes" active="no"/>
@@
 <part name="R4" library="resistor" library_urn="urn:adsk.eagle:library:348" deviceset="R-US_" device="0207/10" package3d_urn="urn:adsk.eagle:package:25939/1" value="2k"/>
 <part name="X_6" library="ngspice-simulation" library_urn="urn:adsk.eagle:library:527439" deviceset="GND" device=""/>
-<part name="R5" library="resistor" library_urn="urn:adsk.eagle:library:348" deviceset="R-US_" device="0207/10" package3d_urn="urn:adsk.eagle:package:25939/1" value="1k"/>
+<part name="R5" library="resistor" library_urn="urn:adsk.eagle:library:348" deviceset="R-US_" device="0207/10" package3d_urn="urn:adsk.eagle:package:25939/1" value="10"/>
 <part name="JP7" library="SparkFun" deviceset="M02" device="PTH4" value="SHIELD_PWR"/>
 <part name="U3" library="SparkFun" deviceset="ARDUINO_SHIELD" device="LABEL"/>
@@
 </instance>
 <instance part="JP2" gate="G$1" x="-132.08" y="53.34" smashed="yes" rot="R180">
-<attribute name="NAME" x="-125.73" y="47.625" size="1.778" layer="95" rot="R180"/>
+<attribute name="NAME" x="-128.27" y="60.325" size="1.778" layer="95" rot="R180"/>
 <attribute name="VALUE" x="-125.73" y="58.42" size="1.778" layer="96" rot="R180"/>
 </instance>

Commit message: Ready to mill
Parts:
- added KK1: SK129-PAD, heatsink:SK129-PAD
Changed lines of the file:
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@@
 <part name="C2" library="rcl" library_urn="urn:adsk.eagle:library:334" deviceset="C-US" device="025-025X050" package3d_urn="urn:adsk.eagle:package:23629/2" value="100n"/>
 <part name="PI" library="raspberrypi_bastelstube_v13" deviceset="RASPI_BOARD_B+" device="_F" value="RASPI_BOARD_B+_F"/>
+<part name="KK1" library="heatsink" library_urn="urn:adsk.eagle:library:236" deviceset="SK129-PAD" device="" package3d_urn="urn:adsk.eagle:package:14199/1"/>
 </parts>
 <sheets>
@@
 </instance>
 <instance part="PI" gate="G$1" x="-48.26" y="7.62" smashed="yes"/>
+<instance part="KK1" gate="G$1" x="-96.52" y="53.34" smashed="yes">
+<attribute name="NAME" x="-90.805" y="56.515" size="1.778" layer="95"/>
+<attribute name="VALUE" x="-90.805" y="53.975" size="1.778" layer="96"/>
+</instance>
 </instances>
 <busses>

Commit message: add blinker LED
Parts:
- added LED3: (no value), led:LED5MM
- added R6: 100, resistor:R-US_0207/10
Connections:
- new net N$4: LED3.A, PI.GPIO25
- new net N$6: LED3.C, R6.2
- net 0: now also R6.1
Changed lines of the file:
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@@
 <part name="PI" library="raspberrypi_bastelstube_v13" deviceset="RASPI_BOARD_B+" device="_F" value="RASPI_BOARD_B+_F"/>
 <part name="KK1" library="heatsink" library_urn="urn:adsk.eagle:library:236" deviceset="SK129-PAD" device="" package3d_urn="urn:adsk.eagle:package:14199/1"/>
+<part name="LED3" library="led" library_urn="urn:adsk.eagle:library:259" deviceset="LED" device="5MM" package3d_urn="urn:adsk.eagle:package:15799/2"/>
+<part name="R6" library="resistor" library_urn="urn:adsk.eagle:library:348" deviceset="R-US_" device="0207/10" package3d_urn="urn:adsk.eagle:package:25939/1" value="100"/>
+<part name="X_3" library="ngspice-simulation" library_urn="urn:adsk.eagle:library:527439" deviceset="GND" device=""/>
 </parts>
 <sheets>
@@
 <attribute name="VALUE" x="-90.805" y="53.975" size="1.778" layer="96"/>
 </instance>
+<instance part="LED3" gate="G$1" x="-93.98" y="-25.4" smashed="yes">
+<attribute name="NAME" x="-90.424" y="-29.972" size="1.778" layer="95" rot="R90"/>
+<attribute name="VALUE" x="-88.265" y="-29.972" size="1.778" layer="96" rot="R90"/>
+</instance>
+<instance part="R6" gate="G$1" x="-93.98" y="-40.64" smashed="yes" rot="R90">
+<attribute name="NAME" x="-95.4786" y="-44.45" size="1.778" layer="95" rot="R90"/>
+<attribute name="VALUE" x="-90.678" y="-44.45" size="1.778" layer="96" rot="R90"/>
+</instance>
+<instance part="X_3" gate="G$1" x="-93.98" y="-50.8" smashed="yes"/>
 </instances>
 <busses>
@@
 <portref moduleinst="TXS0108E1" port="GND"/>
 <wire x1="-88.9" y1="-91.44" x2="-83.82" y2="-91.44" width="0.1524" layer="91"/>
+</segment>
+<segment>
+<pinref part="X_3" gate="G$1" pin="0"/>
+<pinref part="R6" gate="G$1" pin="1"/>
+<wire x1="-93.98" y1="-50.8" x2="-93.98" y2="-45.72" width="0.1524" layer="91"/>
 </segment>
 </net>
@@
 </segment>
 </net>
+<net name="N$4" class="0">
+<segment>
+<pinref part="PI" gate="G$1" pin="GPIO25"/>
+<pinref part="LED3" gate="G$1" pin="A"/>
+<wire x1="-63.5" y1="7.62" x2="-93.98" y2="7.62" width="0.1524" layer="91"/>
+<wire x1="-93.98" y1="7.62" x2="-93.98" y2="-22.86" width="0.1524" layer="91"/>
+</segment>
+</net>
+<net name="N$6" class="0">
+<segment>
+<pinref part="LED3" gate="G$1" pin="C"/>
+<pinref part="R6" gate="G$1" pin="2"/>
+<wire x1="-93.98" y1="-30.48" x2="-93.98" y2="-35.56" width="0.1524" layer="91"/>
+</segment>
+</net>

Commit message: git
Parts:
- added S1: (no value), switch1:MS243
Connections:
- new net N$3: JP2.1, S1.P
- net 0: now also S1.S; no longer JP2.1
Changed lines of the file:
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@@
 <part name="R6" library="resistor" library_urn="urn:adsk.eagle:library:348" deviceset="R-US_" device="0207/10" package3d_urn="urn:adsk.eagle:package:25939/1" value="100"/>
 <part name="X_3" library="ngspice-simulation" library_urn="urn:adsk.eagle:library:527439" deviceset="GND" device=""/>
+<part name="S1" library="switch1" deviceset="MS243" device="" package3d_urn="urn:adsk.eagle:package:27683/1"/>
 </parts>
 <sheets>
@@
 </instance>
 <instance part="X_3" gate="G$1" x="-93.98" y="-50.8" smashed="yes"/>
+<instance part="S1" gate="1" x="-127" y="40.64" smashed="yes" rot="R180">
+<attribute name="NAME" x="-123.19" y="37.465" size="1.778" layer="95" rot="R270"/>
+<attribute name="VALUE" x="-125.73" y="37.465" size="1.778" layer="96" rot="R270"/>
+</instance>
 </instances>
 <busses>
@@
 <net name="0" class="0">
 <segment>
-<pinref part="JP2" gate="G$1" pin="1"/>
-<wire x1="-129.54" y1="50.8" x2="-119.38" y2="45.72" width="0.1524" layer="91"/>
 <pinref part="IC1" gate="A1" pin="GND"/>
-<wire x1="-119.38" y1="45.72" x2="-116.84" y2="45.72" width="0.1524" layer="91"/>
 <pinref part="X_1" gate="G$1" pin="0"/>
 <wire x1="-116.84" y1="45.72" x2="-109.22" y2="45.72" width="0.1524" layer="91"/>
@@
 <junction x="-109.22" y="45.72"/>
 <pinref part="C1" gate="G$1" pin="2"/>
-<junction x="-116.84" y="45.72"/>
 <pinref part="C2" gate="G$1" pin="2"/>
 <wire x1="-83.82" y1="45.72" x2="-96.52" y2="45.72" width="0.1524" layer="91"/>
 <junction x="-96.52" y="45.72"/>
+<wire x1="-116.84" y1="45.72" x2="-116.84" y2="33.02" width="0.1524" layer="91"/>
+<junction x="-116.84" y="45.72"/>
+<pinref part="S1" gate="1" pin="S"/>
+<wire x1="-116.84" y1="33.02" x2="-129.54" y2="33.02" width="0.1524" layer="91"/>
+<wire x1="-129.54" y1="33.02" x2="-129.54" y2="35.56" width="0.1524" layer="91"/>
 </segment>
 <segment>
@@
 </segment>
 </net>
+<net name="N$3" class="0">
+<segment>
+<pinref part="S1" gate="1" pin="P"/>
+<pinref part="JP2" gate="G$1" pin="1"/>
+<wire x1="-129.54" y1="45.72" x2="-129.54" y2="50.8" width="0.1524" layer="91"/>
+</segment>
+</net>

Commit message: fixed switch position
Parts:
- removed S1: (no value), switch1:MS243
- added S2: (no value), switch1:MS243
Connections:
- removed net N$3: JP2.1, S1.P
- new net N$7: JP7.2, S2.P
- net 0: now also JP2.1, S2.S; no longer JP7.2, S1.S
Changed lines of the file:
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@@
 <part name="JP7" library="SparkFun" deviceset="M02" device="PTH4" value="SHIELD_PWR"/>
 <part name="U3" library="SparkFun" deviceset="ARDUINO_SHIELD" device="LABEL"/>
-<part name="X_7" library="ngspice-simulation" library_urn="urn:adsk.eagle:library:527439" deviceset="GND" device=""/>
 <part name="X_9" library="ngspice-simulation" library_urn="urn:adsk.eagle:library:527439" deviceset="GND" device=""/>
 <part name="X_8" library="ngspice-simulation" library_urn="urn:adsk.eagle:library:527439" deviceset="GND" device=""/>
@@
 <part name="R6" library="resistor" library_urn="urn:adsk.eagle:library:348" deviceset="R-US_" device="0207/10" package3d_urn="urn:adsk.eagle:package:25939/1" value="100"/>
 <part name="X_3" library="ngspice-simulation" library_urn="urn:adsk.eagle:library:527439" deviceset="GND" device=""/>
-<part name="S1" library="switch1" deviceset="MS243" device="" package3d_urn="urn:adsk.eagle:package:27683/1"/>
+<part name="S2" library="switch1" deviceset="MS243" device="" package3d_urn="urn:adsk.eagle:package:27683/1"/>
+<part name="X_7" library="ngspice-simulation" library_urn="urn:adsk.eagle:library:527439" deviceset="GND" device=""/>
 </parts>
 <sheets>
@@
 <attribute name="VALUE" x="-39.37" y="-101.6" size="1.778" layer="96" rot="MR0"/>
 </instance>
-<instance part="X_7" gate="G$1" x="5.08" y="-78.74" smashed="yes"/>
 <instance part="X_9" gate="G$1" x="-33.02" y="-104.14" smashed="yes"/>
 <instance part="X_8" gate="G$1" x="-81.28" y="-99.06" smashed="yes"/>
@@
 </instance>
 <instance part="X_3" gate="G$1" x="-93.98" y="-50.8" smashed="yes"/>
-<instance part="S1" gate="1" x="-127" y="40.64" smashed="yes" rot="R180">
-<attribute name="NAME" x="-123.19" y="37.465" size="1.778" layer="95" rot="R270"/>
-<attribute name="VALUE" x="-125.73" y="37.465" size="1.778" layer="96" rot="R270"/>
-</instance>
+<instance part="S2" gate="1" x="7.62" y="-83.82" smashed="yes" rot="R180">
+<attribute name="NAME" x="11.43" y="-86.995" size="1.778" layer="95" rot="R270"/>
+<attribute name="VALUE" x="8.89" y="-86.995" size="1.778" layer="96" rot="R270"/>
+</instance>
+<instance part="X_7" gate="G$1" x="5.08" y="-96.52" smashed="yes"/>
 </instances>
 <busses>
@@
 <wire x1="-83.82" y1="45.72" x2="-96.52" y2="45.72" width="0.1524" layer="91"/>
 <junction x="-96.52" y="45.72"/>
-<wire x1="-116.84" y1="45.72" x2="-116.84" y2="33.02" width="0.1524" layer="91"/>
+<wire x1="-129.54" y1="35.56" x2="-129.54" y2="33.02" width="0.1524" layer="91"/>
+<wire x1="-129.54" y1="33.02" x2="-129.54" y2="30.48" width="0.1524" layer="91"/>
+<wire x1="-129.54" y1="30.48" x2="-116.84" y2="30.48" width="0.1524" layer="91"/>
+<wire x1="-116.84" y1="30.48" x2="-116.84" y2="45.72" width="0.1524" layer="91"/>
 <junction x="-116.84" y="45.72"/>
-<pinref part="S1" gate="1" pin="S"/>
-<wire x1="-116.84" y1="33.02" x2="-129.54" y2="33.02" width="0.1524" layer="91"/>
-<wire x1="-129.54" y1="33.02" x2="-129.54" y2="35.56" width="0.1524" layer="91"/>
+<pinref part="JP2" gate="G$1" pin="1"/>
+<wire x1="-129.54" y1="50.8" x2="-129.54" y2="35.56" width="0.1524" layer="91"/>
 </segment>
 <segment>
@@
 <pinref part="R5" gate="G$1" pin="1"/>
 <wire x1="-129.54" y1="-27.94" x2="-129.54" y2="-25.4" width="0.1524" layer="91"/>
-</segment>
-<segment>
-<pinref part="JP7" gate="G$1" pin="2"/>
-<pinref part="X_7" gate="G$1" pin="0"/>
-<wire x1="-15.24" y1="-76.2" x2="5.08" y2="-76.2" width="0.1524" layer="91"/>
-<wire x1="5.08" y1="-76.2" x2="5.08" y2="-78.74" width="0.1524" layer="91"/>
 </segment>
 <segment>
@@
 <pinref part="R6" gate="G$1" pin="1"/>
 <wire x1="-93.98" y1="-50.8" x2="-93.98" y2="-45.72" width="0.1524" layer="91"/>
+</segment>
+<segment>
+<pinref part="S2" gate="1" pin="S"/>
+<pinref part="X_7" gate="G$1" pin="0"/>
+<wire x1="5.08" y1="-88.9" x2="5.08" y2="-96.52" width="0.1524" layer="91"/>
 </segment>
 </net>
@@
 </segment>
 </net>
-<net name="N$3" class="0">
-<segment>
-<pinref part="S1" gate="1" pin="P"/>
-<pinref part="JP2" gate="G$1" pin="1"/>
-<wire x1="-129.54" y1="45.72" x2="-129.54" y2="50.8" width="0.1524" layer="91"/>
-</segment>
-</net>
+<net name="N$7" class="0">
+<segment>
+<pinref part="JP7" gate="G$1" pin="2"/>
+<wire x1="-15.24" y1="-76.2" x2="5.08" y2="-76.2" width="0.1524" layer="91"/>
+<wire x1="5.08" y1="-76.2" x2="5.08" y2="-78.74" width="0.1524" layer="91"/>
+<pinref part="S2" gate="1" pin="P"/>
+</segment>
+</net>
