File: EAGLE/projects/Bot/bot_display.sch (EAGLE design)
At the start: 16 parts, among them IC1 7805T, U3 ARDUINO_SHIELDLABEL, X1 RASPI_GPIO_B+_PIN

Commit message: revert eagle files
Parts:
- removed JP2: (no value), pinhead:PINHD-1X2
- removed JP7: SHIELD_PWR, SparkFun:M02PTH4
- removed U3: ARDUINO_SHIELDLABEL, SparkFun:ARDUINO_SHIELDLABEL
- removed X1: RASPI_GPIO_B+_PIN, raspberrypi_bastelstube_v13:RASPI_GPIO_B+_PIN
- added BAT1: 11.1V, special:BATTERY
- added M1, M2: MOTOR10MM, SparkFun-Electromechanical:MOTOR10MM
Connections:
- removed net B1: JP2.9
- removed net B2: JP2.8
- removed net B3: JP2.7
- removed net B4: JP2.6
- removed net B5: JP2.5
- removed net B6: JP2.4
- removed net B7: JP2.3
- removed net B8: JP2.2
- removed net GND: JP2.1
- removed net L_BCK: X1.GPIO21
- removed net L_FWD: X1.GPIO20
- removed net L_SPD: U3.*D5, X1.GPIO12
- removed net N$13: U3.D4
- removed net N$14: U3.D7
- removed net N$15: U3.D8
- removed net N$16: U3.*D9
- removed net PI_3V3: X1.3V3
- removed net R_BCK: X1.GPIO06
- removed net R_FWD: X1.GPIO05
- removed net R_SPD: U3.*D6, X1.GPIO13
- removed net R_US_TRIG: U$2.TRIG, X1.GPIO27
- removed net VB: JP2.10
- new net N$3: M1.+
- new net N$4: M1.-
- new net N$6: M2.+
- new net N$7: M2.-
- net 0: now also BAT1.-; no longer JP2.1, JP7.2, U3.GND@0, U3.GND@1, U3.GND@2, X1.GND
- net L_US_ECHO: no longer X1.GPIO24
- net L_US_TRIG: now also U$2.TRIG; no longer X1.GPIO23
- net PI_5V: no longer U3.5V, U3.A0, U3.A1, X1.5V0
- net PWR+: now also BAT1.+; no longer JP2.2, JP7.1
- net R_US_ECHO: no longer X1.GPIO22
Other:
- note removed: "PWR +"
- note removed: "PWR -"
- moved on the sheet: C1, C2, IC1, LED1, LED2, R1, R2, R3, R4, R5, U$1, U$2

Commit message: more restructuring
Parts:
- added LED3: (no value), led:LED5MM
- added R6: 10, resistor:R-US_0207/10
- R5: value 1k -> 10
Connections:
- new net N$10: LED3.A
- new net N$11: LED3.C, R6.2
- net 0: now also R6.1
- net PI_5V: now also LED1.A, LED2.A
- net PWR+: no longer LED1.A, LED2.A
Other:
- moved on the sheet: BAT1, C1, C2, IC1, R1, R2, R3, R4, U$1, U$2

Commit message: add bot_display update
Parts:
- added S1: (no value), switch:MS243
Connections:
- new net N$12: BAT1.+, S1.P
- net PWR+: now also S1.S; no longer BAT1.+
Other:
- moved on the sheet: BAT1
Changed lines of the file:
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@@
 <part name="X_9" library="ngspice-simulation" library_urn="urn:adsk.eagle:library:527439" deviceset="GND" device=""/>
 <part name="R6" library="resistor" library_urn="urn:adsk.eagle:library:348" deviceset="R-US_" device="0207/10" package3d_urn="urn:adsk.eagle:package:25939/1" value="10"/>
+<part name="S1" library="switch" library_urn="urn:adsk.eagle:library:380" deviceset="MS243" device="" package3d_urn="urn:adsk.eagle:package:27683/1"/>
 </parts>
 <sheets>
@@
 </instance>
 <instance part="X_2" gate="G$1" x="-35.56" y="45.72" smashed="yes"/>
-<instance part="BAT1" gate="G$1" x="-127" y="50.8" smashed="yes" rot="R270">
-<attribute name="NAME" x="-121.92" y="52.07" size="1.778" layer="95" rot="R270"/>
-<attribute name="VALUE" x="-133.35" y="54.61" size="1.778" layer="96" rot="R270"/>
+<instance part="BAT1" gate="G$1" x="-137.16" y="50.8" smashed="yes" rot="R270">
+<attribute name="NAME" x="-132.08" y="52.07" size="1.778" layer="95" rot="R270"/>
+<attribute name="VALUE" x="-143.51" y="54.61" size="1.778" layer="96" rot="R270"/>
 </instance>
 <instance part="R2" gate="G$1" x="-106.68" y="-38.1" smashed="yes" rot="MR270">
@@
 <attribute name="VALUE" x="-80.518" y="-21.59" size="1.778" layer="96" rot="R90"/>
 </instance>
+<instance part="S1" gate="1" x="-121.92" y="58.42" smashed="yes" rot="R270">
+<attribute name="NAME" x="-118.745" y="62.23" size="1.778" layer="95"/>
+<attribute name="VALUE" x="-118.745" y="59.69" size="1.778" layer="96"/>
+</instance>
 </instances>
 <busses>
@@
 <pinref part="C1" gate="G$1" pin="1"/>
 <wire x1="-106.68" y1="53.34" x2="-106.68" y2="55.88" width="0.1524" layer="91"/>
-<junction x="-106.68" y="55.88"/>
-<pinref part="BAT1" gate="G$1" pin="+"/>
-<wire x1="-127" y1="55.88" x2="-106.68" y2="55.88" width="0.1524" layer="91"/>
 <wire x1="-106.68" y1="55.88" x2="-96.52" y2="55.88" width="0.1524" layer="91"/>
 <label x="-111.76" y="55.88" size="1.778" layer="95"/>
+<pinref part="S1" gate="1" pin="S"/>
+<wire x1="-106.68" y1="55.88" x2="-116.84" y2="55.88" width="0.1524" layer="91"/>
+<junction x="-106.68" y="55.88"/>
 </segment>
 </net>
@@
 <pinref part="X_1" gate="G$1" pin="0"/>
 <wire x1="-99.06" y1="38.1" x2="-99.06" y2="43.18" width="0.1524" layer="91"/>
+<wire x1="-137.16" y1="43.18" x2="-106.68" y2="43.18" width="0.1524" layer="91"/>
+<junction x="-106.68" y="43.18"/>
 <pinref part="BAT1" gate="G$1" pin="-"/>
-<wire x1="-127" y1="45.72" x2="-127" y2="43.18" width="0.1524" layer="91"/>
-<wire x1="-127" y1="43.18" x2="-106.68" y2="43.18" width="0.1524" layer="91"/>
-<junction x="-106.68" y="43.18"/>
+<wire x1="-137.16" y1="45.72" x2="-137.16" y2="43.18" width="0.1524" layer="91"/>
 </segment>
 <segment>
@@
 <portref moduleinst="RASPBERRY_PI_3B+" port="GPIO20"/>
 <wire x1="-63.5" y1="-10.16" x2="-78.74" y2="-10.16" width="0.1524" layer="91"/>
+<junction x="-78.74" y="-10.16"/>
 </segment>
 <segment>
@@
 <wire x1="-106.68" y1="-96.52" x2="-109.22" y2="-96.52" width="0.1524" layer="91"/>
 <wire x1="-109.22" y1="-96.52" x2="-111.76" y2="-96.52" width="0.1524" layer="91"/>
+<junction x="-111.76" y="-96.52"/>
 </segment>
 </net>
@@
 <portref moduleinst="RASPBERRY_PI_3B+" port="GPIO21"/>
 <wire x1="-63.5" y1="-12.7" x2="-78.74" y2="-12.7" width="0.1524" layer="91"/>
+<junction x="-78.74" y="-12.7"/>
 </segment>
 <segment>
@@
 <wire x1="-96.52" y1="-99.06" x2="-111.76" y2="-99.06" width="0.1524" layer="91"/>
 <label x="-109.22" y="-99.06" size="1.778" layer="95"/>
+<junction x="-111.76" y="-99.06"/>
 </segment>
 </net>
@@
 <portref moduleinst="RASPBERRY_PI_3B+" port="GPIO05"/>
 <wire x1="-63.5" y1="7.62" x2="-78.74" y2="7.62" width="0.1524" layer="91"/>
+<junction x="-78.74" y="7.62"/>
 </segment>
 <segment>
@@
 <wire x1="-96.52" y1="-88.9" x2="-111.76" y2="-88.9" width="0.1524" layer="91"/>
 <label x="-109.22" y="-88.9" size="1.778" layer="95"/>
+<junction x="-111.76" y="-88.9"/>
 </segment>
 </net>
@@
 <portref moduleinst="RASPBERRY_PI_3B+" port="GPIO06"/>
 <wire x1="-63.5" y1="5.08" x2="-78.74" y2="5.08" width="0.1524" layer="91"/>
+<junction x="-78.74" y="5.08"/>
 </segment>
 <segment>
@@
 <wire x1="-96.52" y1="-101.6" x2="-111.76" y2="-101.6" width="0.1524" layer="91"/>
 <label x="-109.22" y="-101.6" size="1.778" layer="95"/>
+<junction x="-111.76" y="-101.6"/>
 </segment>
 </net>
@@
 <portref moduleinst="RASPBERRY_PI_3B+" port="GPIO12"/>
 <wire x1="-63.5" y1="2.54" x2="-78.74" y2="2.54" width="0.1524" layer="91"/>
+<junction x="-78.74" y="2.54"/>
 </segment>
 <segment>
@@
 <label x="-55.88" y="-91.44" size="1.778" layer="95"/>
 <portref moduleinst="MONSTER_MOTO_SHIELD" port="D5"/>
+<junction x="-58.42" y="-91.44"/>
 </segment>
 </net>
@@
 <portref moduleinst="RASPBERRY_PI_3B+" port="GPIO13"/>
 <wire x1="-63.5" y1="0" x2="-78.74" y2="0" width="0.1524" layer="91"/>
+<junction x="-78.74" y="0"/>
 </segment>
 <segment>
@@
 <label x="-55.88" y="-93.98" size="1.778" layer="95"/>
 <portref moduleinst="MONSTER_MOTO_SHIELD" port="D6"/>
+<junction x="-58.42" y="-93.98"/>
 </segment>
 </net>
@@
 <label x="-111.76" y="2.54" size="1.778" layer="95"/>
 <pinref part="U$1" gate="G$1" pin="TRIG"/>
+<junction x="-88.9" y="2.54"/>
 </segment>
 <segment>
@@
 <label x="-111.76" y="-50.8" size="1.778" layer="95"/>
 <pinref part="U$2" gate="G$1" pin="TRIG"/>
+<junction x="-88.9" y="-50.8"/>
 </segment>
 </net>
@@
 <wire x1="-106.68" y1="-30.48" x2="-88.9" y2="-30.48" width="0.1524" layer="91"/>
 <junction x="-106.68" y="-30.48"/>
+<junction x="-88.9" y="-30.48"/>
 </segment>
 </net>
@@
 </segment>
 </net>
+<net name="N$12" class="0">
+<segment>
+<pinref part="BAT1" gate="G$1" pin="+"/>
+<pinref part="S1" gate="1" pin="P"/>
+<wire x1="-137.16" y1="55.88" x2="-127" y2="55.88" width="0.1524" layer="91"/>
+</segment>
+</net>
