File: EAGLE/projects/Bot/ECD.sch (EAGLE design)
At the start: 20 parts, among them IC2 7805T, U3 ARDUINO_SHIELDLABEL

Commit message: ECD
Parts:
- removed IC2: 7805T, linear:7805T
- removed JP2: (no value), pinhead:PINHD-1X2
- removed JP7: SHIELD_PWR, SparkFun:M02PTH4
- removed KK1: SK129-PAD, heatsink:SK129-PAD
- removed LED1, LED2, LED3: (no value), ledMe:LED5MM
- removed PI: RASPI_BOARD_B+_F, raspberrypi_bastelstube_v13:RASPI_BOARD_B+_F
- removed S2: (no value), switch2:MS243
- removed U$1, U$2: ULTRASONIC-HC-SR04, diy-modules:ULTRASONIC-HC-SR04
- removed U3: ARDUINO_SHIELDLABEL, SparkFun:ARDUINO_SHIELDLABEL
- added IC1: 7805T, linear:7805T
- R6: value 100 -> 10
Connections:
- removed net B1: JP2.9
- removed net B2: JP2.8
- removed net B3: JP2.7
- removed net B4: JP2.6
- removed net B5: JP2.5
- removed net B6: JP2.4
- removed net B7: JP2.3
- removed net B8: JP2.2
- removed net GND: JP2.1
- removed net L_BCK: PI.GPIO21
- removed net L_FWD: PI.GPIO20
- removed net L_SPD: PI.GPIO12, U3.*D5
- removed net L_US_TRIG: PI.GPIO23, U$1.TRIG
- removed net N$1: R1.2, U$1.ECHO
- removed net N$13: U3.D4
- removed net N$14: U3.D7
- removed net N$15: U3.D8
- removed net N$16: U3.*D9
- removed net N$2: R2.2, U$2.ECHO
- removed net N$5: LED1.C, LED2.C, R5.2
- removed net N$6: LED3.C, R6.2
- removed net N$7: JP7.2, S2.P
- removed net PI_3V3: PI.3V3
- removed net PWR+: C1.1, IC2.VI, JP2.2, JP7.1
- removed net R_BCK: PI.GPIO06
- removed net R_FWD: PI.GPIO05
- removed net R_SPD: PI.GPIO13, U3.*D6
- removed net R_US_TRIG: PI.GPIO27, U$2.TRIG
- removed net VB: JP2.10
- new net BAT-: C1.2, C2.2, IC1.GND
- new net LED3_CATHODE: R6.2
- new net L_US_GND: R3.2
- new net R_US_GND: R4.2
- new net S1+: C1.1, IC1.VI
- net 0: no longer C1.2, C2.2, IC2.GND, JP2.1, PI.GND, R3.2, R4.2, S2.S, U$1.GND, U$2.GND, U3.GND@0, U3.GND@1, U3.GND@2
- net L_US_ECHO: now also R1.2; no longer PI.GPIO24
- net N$4: now also R5.2; no longer LED3.A, PI.GPIO25
- net PI_5V: now also IC1.VO; no longer IC2.VO, LED1.A, LED2.A, PI.5V0, U$1.VCC, U$2.VCC, U3.5V, U3.A0, U3.A1
- net R_US_ECHO: now also R2.2; no longer PI.GPIO22
Other:
- note removed: "PWR +"
- note removed: "PWR -"
- moved on the sheet: C1, C2, R1, R2, R3, R4, R5, R6
